File: minipro4/Teilentwurf.brd (EAGLE design)
At the start: 105.1 x 94.6 mm, 62 parts, among them IC1 MEGA8-P, IC2 FT232RL_ADAPTER, IC3 78L08Z, IC4 4051N, J1 HOHLSTECKER, Q2 BS170, Q3 BS170, Q4 BS170, Q6 IRF4905, X1 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

Commit message: < ‘minipro4/Teilentwurf.b##’ > ‘minipro4/Teilentwurf.b#1’ / ‘minipro4/Teilentwurf.brd’ < ‘minipro4/Teilentwurf.s##’ > ‘minipro4/Teilentwurf.s#1’ / ‘minipro4/Teilentwurf.sch’
Parts:
- added C17: (no value), 03_device-library:C025-030X050
- added IC5, IC7: TL082P, 03_device-library:DIL08
- added IC6: 4051N, 03_device-library:DIL16
- added R15, R21: 10k, 03_device-library:0207/10
- added R16, R17, R18, R22, R23, R24, R25: 100k, 03_device-library:0207/10
- added R19, R20: 15k, 03_device-library:0207/10
- added R26: (no value), 03_device-library:POT
- added R27: (no value), 03_device-library:0207/10
- added R28: 8k2, 03_device-library:0207/10
- added R32: 220, 03_device-library:0207/10
Connections:
- new net N$25: IC4.3, IC5.3
- new net N$26: IC5.2, IC6.3
- new net N$27: IC5.5, R22.1, R23.2
- new net N$28: R19.1, R20.2
- new net N$31: IC6.13, R15.1, R21.2
- new net N$32: IC6.14, R15.2, R20.1
- new net N$33: IC6.15, R17.1, R18.1, R19.2
- new net N$34: IC5.1, R16.2, R22.2
- new net N$35: IC5.7, IC7.5, R24.1
- new net N$36: IC5.6, R24.2, R25.1
- new net N$37: IC7.1, IC7.2, R25.2
- new net N$38: R26.3, R27.2
- new net N$39: IC7.3, R26.2
- new net N$40: IC7.6, IC7.7, R28.1
- new net N$41: R28.2, R32.1
- new net N$42: C17.1, R32.2
- net GND: now also C17.2, IC6.8, R21.1, R23.1
- net MUX0*: now also IC6.1, IC6.11, IC6.12, IC6.2, IC6.4, IC6.5, R16.1, R17.2, R18.2
- net MUX1*: now also IC6.10
- net MUX2*: now also IC6.9
- net V+: now also IC5.8, IC6.16, IC7.8, R27.1
- net V-: now also IC5.4, IC6.7, IC7.4, R26.1

Commit message: / ‘minipro4/Teilentwurf.b#1’ < ‘minipro4/Teilentwurf.b##’ > ‘minipro4/Teilentwurf.b#2’ / ‘minipro4/Teilentwurf.brd’ / ‘minipro4/Teilentwurf.s#1’ < ‘minipro4/Teilentwurf.s##’ > ‘minipro4/Teilentwurf.s#2’ / ‘minipro4/Teilentwurf.sch’
Parts:
- C8: value (none) -> 1uF
- R10, R12: value (none) -> 1M
- R11, R13, R14, R6, R7: value (none) -> 100k
- R27: value (none) -> 22k
- R8: value (none) -> 120k
- R9: value (none) -> 180k
Connections:
- net V+: now also R26.1; no longer R27.1
- net V-: now also R27.1; no longer R26.1
Changed lines of the file:
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@@
 <element name="R2" library="03_device-library" package="0207/10" value="4.7k" x="17.145" y="79.375" rot="R180"/>
 <element name="R5" library="03_device-library" package="0207/10" value="10k" x="12.065" y="76.835"/>
-<element name="R6" library="03_device-library" package="0207/10" value="" x="-5.08" y="-6.35"/>
-<element name="R7" library="03_device-library" package="0207/10" value="" x="-5.08" y="-11.43"/>
-<element name="R8" library="03_device-library" package="0207/10" value="" x="-5.08" y="-16.51"/>
-<element name="R9" library="03_device-library" package="0207/10" value="" x="-5.08" y="-21.59"/>
-<element name="R10" library="03_device-library" package="0207/10" value="" x="-5.08" y="-26.67"/>
-<element name="R11" library="03_device-library" package="0207/10" value="" x="-5.08" y="-31.75"/>
-<element name="R12" library="03_device-library" package="0207/10" value="" x="-5.08" y="-36.83"/>
-<element name="R13" library="03_device-library" package="0207/10" value="" x="-5.08" y="-41.91"/>
-<element name="R14" library="03_device-library" package="0207/10" value="" x="-5.08" y="-46.99"/>
+<element name="R6" library="03_device-library" package="0207/10" value="100k" x="-5.08" y="-6.35"/>
+<element name="R7" library="03_device-library" package="0207/10" value="100k" x="-5.08" y="-11.43"/>
+<element name="R8" library="03_device-library" package="0207/10" value="120k" x="-5.08" y="-16.51"/>
+<element name="R9" library="03_device-library" package="0207/10" value="180k" x="-5.08" y="-21.59"/>
+<element name="R10" library="03_device-library" package="0207/10" value="1M" x="-5.08" y="-26.67"/>
+<element name="R11" library="03_device-library" package="0207/10" value="100k" x="-5.08" y="-31.75"/>
+<element name="R12" library="03_device-library" package="0207/10" value="1M" x="-5.08" y="-36.83"/>
+<element name="R13" library="03_device-library" package="0207/10" value="100k" x="-5.08" y="-41.91"/>
+<element name="R14" library="03_device-library" package="0207/10" value="100k" x="-5.08" y="-46.99"/>
 <element name="IC4" library="03_device-library" package="DIL16" value="4051N" x="1.27" y="-54.61"/>
 <element name="S1" library="03_device-library" package="APEM_5236" value="SWITCH" x="-20.32" y="-49.53"/>
-<element name="C8" library="03_device-library" package="C050-050X075" value="" x="-20.32" y="-66.04"/>
+<element name="C8" library="03_device-library" package="C050-050X075" value="1uF" x="-20.32" y="-66.04"/>
 <element name="X2" library="03_device-library" package="CON_COAX" value="CON_COAX" x="8.89" y="-77.47"/>
 <element name="IC5" library="03_device-library" package="DIL08" value="TL082P" x="-16.51" y="-91.44"/>
@@
 <element name="R25" library="03_device-library" package="0207/10" value="100k" x="-17.78" y="-177.8"/>
 <element name="R26" library="03_device-library" package="POT" value="" x="8.89" y="-186.69"/>
-<element name="R27" library="03_device-library" package="0207/10" value="" x="-17.78" y="-198.12"/>
+<element name="R27" library="03_device-library" package="0207/10" value="22k" x="-17.78" y="-198.12"/>
 <element name="R28" library="03_device-library" package="0207/10" value="8k2" x="-17.78" y="-203.2"/>
 <element name="R32" library="03_device-library" package="0207/10" value="220" x="-17.78" y="-208.28"/>
@@
 <contactref element="IC6" pad="16"/>
 <contactref element="IC7" pad="8"/>
-<contactref element="R27" pad="1"/>
-<wire x1="-20.32" y1="-163.83" x2="-22.86" y2="-198.12" width="0" layer="19" extent="1-1"/>
+<contactref element="R26" pad="1"/>
+<wire x1="7.62" y1="-181.61" x2="-20.32" y2="-163.83" width="0" layer="19" extent="1-1"/>
 <wire x1="-20.32" y1="-100.33" x2="-20.32" y2="-163.83" width="0" layer="19" extent="1-1"/>
 <wire x1="-20.32" y1="-87.63" x2="-20.32" y2="-100.33" width="0" layer="19" extent="1-1"/>
@@
 <contactref element="IC6" pad="7"/>
 <contactref element="IC7" pad="4"/>
-<contactref element="R26" pad="1"/>
-<wire x1="7.62" y1="-181.61" x2="-12.7" y2="-171.45" width="0" layer="19" extent="1-1"/>
+<contactref element="R27" pad="1"/>
+<wire x1="-12.7" y1="-171.45" x2="-22.86" y2="-198.12" width="0" layer="19" extent="1-1"/>
 <wire x1="-5.08" y1="-107.95" x2="-12.7" y2="-171.45" width="0" layer="19" extent="1-1"/>
 <wire x1="-12.7" y1="-95.25" x2="-5.08" y2="-107.95" width="0" layer="19" extent="1-1"/>

Commit message: nvdsjbjisd
Parts:
- C17: value (none) -> 1nF
- R26: value (none) -> 100k
- moved C17 272.1 mm to (96.5, 31.8)
- moved R32 261.8 mm to (97.8, 26.7), turned to 180 degrees
- moved R28 252.8 mm to (97.8, 21.6)
- moved R27 231.4 mm to (95.2, 3.81), turned to 180 degrees
- moved R21 216.5 mm to (85.1, 45.7), turned to 90 degrees
- moved R25 213.0 mm to (63.5, 19.1)
- moved IC7 210.4 mm to (94.0, 11.4), turned to 270 degrees
- moved R20 209.6 mm to (80.0, 45.7), turned to 90 degrees
- moved R26 204.1 mm to (78.7, 5.08), turned to 90 degrees
- moved R19 203.9 mm to (77.5, 45.7), turned to 270 degrees
- moved R18 197.1 mm to (72.4, 45.7), turned to 90 degrees
- moved R24 192.8 mm to (59.7, 16.5), turned to 180 degrees
- moved R22 192.7 mm to (53.3, 29.2), turned to 90 degrees
- moved R17 191.4 mm to (69.8, 45.7), turned to 90 degrees
- moved R15 188.9 mm to (82.5, 45.7), turned to 270 degrees
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Connections:
- removed net N$42: C17.1, R32.2
- net AD+: now also C17.1, R32.2
- net GND: now also IC6.6
- net MUX0*: no longer IC6.1, IC6.12, IC6.2, IC6.4, IC6.5, R16.1, R17.2, R18.2
- net N$13: now also R13.2
- net N$19: now also R12.1
- net N$22: now also R13.1, R14.2
- net N$23: now also IC6.1, IC6.12, IC6.2, IC6.4, IC6.5, R16.1, R17.2, R18.2; no longer R13.1, R14.2
- net N$24: now also R12.2
Routing:
- net GND: track 412.7 -> 452.2 mm, vias 0 -> 1
- net MUX2*: track 24.5 -> 0.00 mm
- net V+: track 14.6 -> 29.0 mm, vias 0 -> 1
- net AD+: track 12.7 -> 0.00 mm
- net MUX1*: track 10.5 -> 0.00 mm
- net N$24: track 0.00 -> 9.42 mm
- net V-: track 18.8 -> 19.5 mm

Commit message: dadsadsaasd
Parts:
- added C18, C19, C20, C21, C22, C23, C24, C25: 100nF, 03_device-library:C025-030X050
Connections:
- net GND: now also C18.2, C19.1
- net V+: now also C18.1
- net V-: now also C19.2
Changed lines of the file:
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@@
 <element name="R32" library="03_device-library" package="0207/10" value="220" x="97.79" y="26.67" rot="R180"/>
 <element name="C17" library="03_device-library" package="C025-030X050" value="1nF" x="96.52" y="31.75"/>
+<element name="C18" library="03_device-library" package="C025-030X050" value="100nF" x="-7.62" y="-33.02"/>
+<element name="C19" library="03_device-library" package="C025-030X050" value="100nF" x="-7.62" y="-39.37"/>
+<element name="C20" library="03_device-library" package="C025-030X050" value="100nF" x="-7.62" y="-45.72"/>
+<element name="C21" library="03_device-library" package="C025-030X050" value="100nF" x="-7.62" y="-52.07"/>
+<element name="C22" library="03_device-library" package="C025-030X050" value="100nF" x="-7.62" y="-58.42"/>
+<element name="C23" library="03_device-library" package="C025-030X050" value="100nF" x="-7.62" y="-64.77"/>
+<element name="C24" library="03_device-library" package="C025-030X050" value="100nF" x="-7.62" y="-71.12"/>
+<element name="C25" library="03_device-library" package="C025-030X050" value="100nF" x="-7.62" y="-77.47"/>
 </elements>
 <signals>
@@
 <via x="88.9" y="45.72" extent="1-16" drill="0.7"/>
 <contactref element="IC6" pad="6"/>
-<wire x1="88.9" y1="45.72" x2="97.79" y2="31.75" width="0" layer="19" extent="1-1"/>
+<contactref element="C18" pad="2"/>
+<contactref element="C19" pad="1"/>
+<wire x1="101.2155" y1="43.18" x2="97.79" y2="31.75" width="0" layer="19" extent="16-16"/>
+<wire x1="85.09" y1="40.64" x2="89.535" y2="43.18" width="0" layer="19" extent="16-16"/>
 <wire x1="58.42" y1="50.8" x2="52.07" y2="52.07" width="0" layer="19" extent="16-16"/>
 <wire x1="60.96" y1="50.8" x2="58.42" y2="50.8" width="0" layer="19" extent="1-1"/>
-<wire x1="85.09" y1="40.64" x2="97.79" y2="31.75" width="0" layer="19" extent="1-1"/>
+<wire x1="31.75" y1="33.02" x2="27.5555" y2="40.005" width="0" layer="19" extent="16-16"/>
+<wire x1="36.83" y1="33.02" x2="31.75" y2="33.02" width="0" layer="19" extent="1-1"/>
 <wire x1="73.66" y1="34.29" x2="85.09" y2="40.64" width="0" layer="19" extent="1-1"/>
 <wire x1="68.58" y1="34.29" x2="73.66" y2="34.29" width="0" layer="19" extent="1-1"/>
-<wire x1="31.75" y1="33.02" x2="27.5555" y2="40.005" width="0" layer="19" extent="16-16"/>
-<wire x1="36.83" y1="33.02" x2="31.75" y2="33.02" width="0" layer="19" extent="1-1"/>
 <wire x1="41.91" y1="6.35" x2="22.86" y2="13.97" width="0" layer="19" extent="16-16"/>
 <wire x1="49.53" y1="11.43" x2="41.91" y2="6.35" width="0" layer="19" extent="1-1"/>
 <wire x1="52.07" y1="6.35" x2="49.53" y2="11.43" width="0" layer="19" extent="1-1"/>
 <wire x1="53.34" y1="20.32" x2="49.53" y2="11.43" width="0" layer="19" extent="1-1"/>
+<wire x1="-6.35" y1="-33.02" x2="9.525" y2="1.905" width="0" layer="19" extent="1-1"/>
+<wire x1="-8.89" y1="-39.37" x2="-6.35" y2="-33.02" width="0" layer="19" extent="1-1"/>
 </signal>
 <signal name="N$20">
@@
 <wire x1="5.715" y1="1.905" x2="5.715" y2="7.62" width="1.016" layer="16"/>
 <contactref element="IC4" pad="16"/>
-<contactref element="IC5" pad="8"/>
 <contactref element="IC6" pad="16"/>
 <contactref element="IC7" pad="8"/>
@@
 <wire x1="5.08" y1="7.62" x2="5.715" y2="7.62" width="1.016" layer="1"/>
 <via x="17.78" y="5.08" extent="1-16" drill="0.7"/>
+<contactref element="C18" pad="1"/>
+<contactref element="IC5" pad="8"/>
 <wire x1="95.885" y1="36.195" x2="100.965" y2="36.195" width="0" layer="19" extent="1-1"/>
 <wire x1="92.075" y1="36.195" x2="95.885" y2="36.195" width="0" layer="19" extent="1-1"/>
@@
 <wire x1="73.66" y1="3.81" x2="63.5" y2="24.13" width="0" layer="19" extent="1-1"/>
 <wire x1="17.78" y1="5.08" x2="49.53" y2="25.4" width="0" layer="19" extent="1-1"/>
+<wire x1="-8.89" y1="-33.02" x2="1.905" y2="1.905" width="0" layer="19" extent="1-1"/>
 </signal>
 <signal name="V-">
@@
 <wire x1="20.32" y1="17.145" x2="21.59" y2="17.145" width="1.016" layer="16"/>
 <contactref element="IC4" pad="7"/>
-<contactref element="IC5" pad="4"/>
 <contactref element="IC6" pad="7"/>
 <contactref element="IC7" pad="4"/>
@@
 <wire x1="21.59" y1="17.145" x2="21.59" y2="23.495" width="1.016" layer="16"/>
 <wire x1="20.32" y1="17.78" x2="20.32" y2="17.145" width="1.016" layer="1"/>
+<contactref element="IC5" pad="4"/>
+<contactref element="C19" pad="2"/>
 <wire x1="55.88" y1="31.75" x2="71.12" y2="34.29" width="0" layer="19" extent="1-1"/>
 <wire x1="34.29" y1="33.02" x2="55.88" y2="31.75" width="0" layer="19" extent="1-1"/>
@@
 <wire x1="90.17" y1="7.62" x2="71.12" y2="34.29" width="0" layer="19" extent="1-1"/>
 <wire x1="100.33" y1="3.81" x2="90.17" y2="7.62" width="0" layer="19" extent="1-1"/>
+<wire x1="-6.35" y1="-39.37" x2="20.32" y2="17.145" width="0" layer="19" extent="16-16"/>
 </signal>
 <signal name="N$4">

Commit message: eagle iteration
Parts:
- moved C8 69.5 mm to (29.2, -53.3), turned to 90 degrees
- moved R28 68.7 mm to (163.8, 2.54)
- moved X2 66.1 mm to (44.5, -54.6)
- moved S1 65.9 mm to (14.0, -57.1)
- moved C17 64.8 mm to (161.3, 34.3)
- moved R32 51.1 mm to (148.6, 21.6)
- moved R8 50.3 mm to (80.0, 8.89), turned to 270 degrees
- moved IC7 44.7 mm to (137.2, 0.00), turned to 90 degrees
- moved R16 42.3 mm to (39.4, 14.0), turned to 180 degrees
- moved R10 41.3 mm to (74.9, 38.1), turned to 0 degrees
- moved R21 41.3 mm to (55.9, 16.5), turned to 270 degrees
- moved R11 41.0 mm to (72.4, 6.35), turned to 180 degrees
- moved R20 39.9 mm to (40.6, 39.4), turned to 180 degrees
- moved R12 39.8 mm to (74.9, 34.3), turned to 180 degrees
- moved R7 39.6 mm to (74.9, 16.5), turned to 180 degrees
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Connections:
- net GND: now also C20.2, C21.1, C22.2, C23.1, C24.2, C25.1
- net V+: now also C20.1, C22.1, C24.1
- net V-: now also C21.2, C23.2, C25.2

Commit message: Layout
Parts:
- added R33: 0, 03_device-library:0207/10
- R28, R32: device 03_device-library:0207/10 -> 03_device-library:0207/15
- moved C25 138.5 mm to (85.1, 25.4), turned to 180 degrees
- moved C24 133.5 mm to (67.3, 39.4), turned to 180 degrees
- moved C23 115.2 mm to (57.1, 30.5), turned to 90 degrees
- moved C22 110.3 mm to (38.1, 41.9), turned to 180 degrees
- moved R28 103.7 mm to (61.0, 15.2), turned to 90 degrees
- moved S1 103.3 mm to (87.6, 15.2), turned to 180 degrees
- moved C20 97.0 mm to (76.8, 1.91), turned to 90 degrees
- moved C21 95.8 mm to (64.1, 11.4), turned to 270 degrees
- moved X2 94.5 mm to (92.7, 26.7), turned to 180 degrees
- moved C8 93.4 mm to (95.2, 12.7), turned to 270 degrees
- moved R32 89.3 mm to (62.2, 44.5), turned to 90 degrees
- moved C19 78.4 mm to (52.1, 11.4), turned to 270 degrees
- moved C17 77.8 mm to (86.4, 55.2), turned to 270 degrees
- moved C18 69.2 mm to (40.6, 16.5), turned to 90 degrees
- moved IC7 68.1 mm to (69.2, 4.45), turned to 180 degrees
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Connections:
- new net N$42: IC6.9, R33.2
- net MUX2*: now also R33.1; no longer IC6.9
- net N$25: now also IC5.5; no longer IC5.3
- net N$26: now also IC5.6; no longer IC5.2
- net N$27: now also IC5.3; no longer IC5.5
- net N$34: now also IC5.7; no longer IC5.1
- net N$35: now also IC5.1; no longer IC5.7
- net N$36: now also IC5.2; no longer IC5.6
Routing:
- net V+: track 29.0 -> 283.0 mm, vias 1 -> 0
- net V-: track 19.5 -> 141.1 mm
- net GND: track 452.2 -> 531.0 mm, vias 1 -> 0
- net AD+: track 0.00 -> 77.8 mm
- net MUX1*: track 0.00 -> 60.0 mm, vias 0 -> 1
- net MUX0*: track 3.81 -> 63.5 mm
- net N$24: track 9.42 -> 59.5 mm, vias 0 -> 1
- net MUX2*: track 0.00 -> 48.9 mm
- net N$39: track 0.00 -> 41.3 mm
- net N$35: track 0.00 -> 39.3 mm
- net N$25: track 0.00 -> 38.2 mm
- net N$23: track 0.00 -> 35.1 mm
- net N$31: track 0.00 -> 34.2 mm
- net N$18: track 0.00 -> 27.7 mm
- net N$38: track 0.00 -> 26.3 mm
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