File: minipro4/Teilentwurf.brd (EAGLE design)
At the start: 105.1 x 94.6 mm, 90 parts, among them IC1 MEGA8-P, IC2 FT232RL_ADAPTER, IC3 78L08Z, IC4 4051N, IC5 TL082P, IC6 4051N, IC7 TL082P, J1 HOHLSTECKER, Q2 BS170, Q3 BS170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

Commit message: Layout Iteration
Parts:
- added R34: 0, 03_device-library:0207/10
- R25: device 03_device-library:0207/10 -> resistor:0207/7
- R28: device 03_device-library:0207/15 -> 03_device-library:0207/10
- moved R21 30.7 mm to (50.8, 50.8), turned to 0 degrees
- moved R25 29.8 mm to (81.0, 5.58), turned to 135 degrees
- moved AD+ 6.75 mm to (66.7, 76.8)
- moved R10 6.48 mm to (78.7, 45.7), turned to 270 degrees
- moved R33 5.68 mm to (83.8, 45.7), turned to 90 degrees
- moved R12 3.42 mm to (75.6, 45.7), turned to 270 degrees
- moved C20 2.83 mm to (76.5, 1.84), turned to 90 degrees
- moved R28 2.54 mm to (58.4, 17.8)
- moved R15 1.27 mm to (50.8, 48.3)
- moved R19 1.27 mm to (38.1, 45.7)
- moved R20 1.27 mm to (38.1, 48.3)
Connections:
- removed net N$42: IC6.9, R33.2
- new net MUX1*A: IC4.10, R33.1
- new net N$45: IC6.11, R34.2
- net MUX0*: now also R34.1; no longer IC6.11
- net MUX1*: now also R33.2; no longer IC4.10
- net MUX2*: now also IC6.9; no longer R33.1
Routing:
- net N$36: track 2.54 -> 46.0 mm
- net MUX0*: track 63.5 -> 26.8 mm
- net N$45: track 0.00 -> 32.4 mm
- net MUX2*: track 48.9 -> 74.3 mm
- net N$42: track 17.0 -> 0.00 mm
- net N$19: track 21.3 -> 36.9 mm
- net N$31: track 26.5 -> 12.3 mm
- net N$37: track 19.8 -> 9.38 mm
- net MUX1*: track 60.0 -> 52.3 mm, vias 1 -> 0
- net N$40: track 15.7 -> 21.9 mm
- net MUX1*A: track 0.00 -> 3.81 mm
- net N$24: track 59.5 -> 55.8 mm, vias 1 -> 0
- net V+: track 279.8 -> 276.3 mm
- net N$39: track 34.0 -> 36.0 mm
- net V-: track 141.1 -> 139.7 mm
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
Commit message: Winkel überarbeitet
Routing:
- net N$23: track 35.3 -> 35.9 mm
Changed lines of the file:
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@@
 </class>
 </classes>
-<designrules name="DesignRules_Grounplane">
+<designrules name="DesignRules_Grounplane *">
 <description language="de">&lt;b&gt;EAGLE Design Rules&lt;/b&gt;
 &lt;p&gt;
@@
 <param name="dpGapFactor" value="2.5"/>
 <param name="checkGrid" value="0"/>
-<param name="checkAngle" value="0"/>
+<param name="checkAngle" value="1"/>
 <param name="checkFont" value="1"/>
 <param name="checkRestrict" value="1"/>
@@
 <contactref element="C17" pad="1"/>
 <wire x1="92.71" y1="67.31" x2="92.71" y2="63.5" width="1.016" layer="1"/>
-<wire x1="62.23" y1="52.07" x2="66.04" y2="55.245" width="1.016" layer="16"/>
 <wire x1="66.04" y1="55.245" x2="83.82" y2="55.245" width="1.016" layer="16"/>
-<wire x1="83.82" y1="55.245" x2="84.455" y2="56.515" width="1.016" layer="16"/>
-<wire x1="84.455" y1="56.515" x2="86.36" y2="56.515" width="1.016" layer="16"/>
 <wire x1="86.36" y1="56.515" x2="86.36" y2="57.15" width="1.016" layer="1"/>
 <wire x1="86.36" y1="57.15" x2="92.71" y2="63.5" width="1.016" layer="1"/>
@@
 <wire x1="69.215" y1="73.025" x2="69.215" y2="76.835" width="1.016" layer="1"/>
 <via x="69.215" y="76.835" extent="1-16" drill="0.8" shape="square"/>
+<wire x1="66.04" y1="55.245" x2="62.865" y2="52.07" width="1.016" layer="16"/>
+<wire x1="62.865" y1="52.07" x2="62.23" y2="52.07" width="1.016" layer="16"/>
+<wire x1="86.36" y1="56.515" x2="85.09" y2="56.515" width="1.016" layer="16"/>
+<wire x1="85.09" y1="56.515" x2="83.82" y2="55.245" width="1.016" layer="16"/>
 </signal>
 <signal name="MUX0">
@@
 <wire x1="56.2645" y1="61.595" x2="53.975" y2="63.8845" width="1.016" layer="16"/>
 <wire x1="53.975" y1="63.8845" x2="53.975" y2="74.5455" width="1.016" layer="16"/>
-<wire x1="53.975" y1="74.5455" x2="56.2645" y2="76.835" width="1.016" layer="16"/>
 <wire x1="78.74" y1="88.9" x2="91.549" y2="88.9" width="1.016" layer="16"/>
 <wire x1="91.549" y1="88.9" x2="93.345" y2="87.104" width="1.016" layer="16"/>
 <wire x1="93.345" y1="87.104" x2="93.345" y2="86.36" width="1.016" layer="16"/>
 <wire x1="56.2645" y1="76.835" x2="56.1975" y2="76.835" width="1.016" layer="16"/>
-<wire x1="56.1975" y1="76.835" x2="58.7375" y2="79.0575" width="1.016" layer="16"/>
-<wire x1="58.7375" y1="79.0575" x2="69.215" y2="79.375" width="1.016" layer="16"/>
 <wire x1="69.215" y1="79.375" x2="78.74" y2="88.9" width="1.016" layer="16"/>
+<wire x1="69.215" y1="79.375" x2="58.8045" y2="79.375" width="1.016" layer="16"/>
+<wire x1="58.8045" y1="79.375" x2="53.975" y2="74.5455" width="1.016" layer="16"/>
+<wire x1="53.975" y1="74.5455" x2="56.1975" y2="76.835" width="0" layer="19" extent="16-16"/>
 </signal>
 <signal name="N$5">
@@
 <contactref element="IC6" pad="10"/>
 <contactref element="R33" pad="2"/>
-<wire x1="57.15" y1="41.91" x2="57.15" y2="42.545" width="1.016" layer="16"/>
-<wire x1="57.15" y1="42.545" x2="59.055" y2="45.085" width="1.016" layer="16"/>
 <wire x1="59.055" y1="45.085" x2="82.55" y2="45.085" width="1.016" layer="16"/>
 <wire x1="82.55" y1="45.085" x2="83.82" y2="46.355" width="1.016" layer="16"/>
 <wire x1="83.82" y1="46.355" x2="83.82" y2="50.8" width="1.016" layer="16"/>
 <wire x1="92.075" y1="46.355" x2="83.82" y2="46.355" width="1.016" layer="16"/>
+<wire x1="57.15" y1="41.91" x2="57.15" y2="43.18" width="1.016" layer="16"/>
+<wire x1="57.15" y1="43.18" x2="59.055" y2="45.085" width="1.016" layer="16"/>
 </signal>
 <signal name="MUX2*">
@@
 <contactref element="IC6" pad="14"/>
 <wire x1="43.18" y1="48.26" x2="45.72" y2="48.26" width="1.016" layer="16"/>
-<wire x1="45.72" y1="48.26" x2="46.99" y2="41.91" width="1.016" layer="16"/>
+<wire x1="46.99" y1="41.91" x2="46.99" y2="46.99" width="1.016" layer="16"/>
+<wire x1="46.99" y1="46.99" x2="45.72" y2="48.26" width="1.016" layer="16"/>
 </signal>
 <signal name="N$33">
@@
 <contactref element="R18" pad="1"/>
 <contactref element="IC6" pad="15"/>
-<wire x1="43.18" y1="45.72" x2="44.45" y2="41.91" width="1.016" layer="16"/>
 <wire x1="40.64" y1="29.21" x2="40.64" y2="26.67" width="1.016" layer="16"/>
 <wire x1="40.64" y1="29.21" x2="40.64" y2="31.75" width="1.016" layer="16"/>
@@
 <wire x1="39.37" y1="35.56" x2="44.45" y2="40.64" width="1.016" layer="16"/>
 <wire x1="44.45" y1="40.64" x2="44.45" y2="41.91" width="1.016" layer="16"/>
+<wire x1="44.45" y1="41.91" x2="44.45" y2="44.45" width="1.016" layer="16"/>
+<wire x1="44.45" y1="44.45" x2="43.18" y2="45.72" width="1.016" layer="16"/>
 </signal>
 <signal name="N$34">
@@
 <wire x1="81.28" y1="12.7" x2="81.28" y2="11.43" width="1.016" layer="16"/>
 <wire x1="81.28" y1="11.43" x2="86.36" y2="6.35" width="1.016" layer="16"/>
-<wire x1="95.25" y1="6.35" x2="101.6" y2="1.27" width="1.016" layer="16"/>
-<wire x1="86.36" y1="6.35" x2="95.25" y2="6.35" width="1.016" layer="16"/>
+<wire x1="86.36" y1="6.35" x2="96.52" y2="6.35" width="1.016" layer="16"/>
+<wire x1="96.52" y1="6.35" x2="101.6" y2="1.27" width="1.016" layer="16"/>
 </signal>
 <signal name="N$39">
@@
 <wire x1="67.945" y1="8.255" x2="67.945" y2="10.16" width="1.016" layer="16"/>
 <wire x1="67.945" y1="10.16" x2="69.215" y2="11.43" width="1.016" layer="16"/>
-<wire x1="96.52" y1="1.27" x2="96.52" y2="2.54" width="1.016" layer="16"/>
-<wire x1="96.52" y1="2.54" x2="94.615" y2="4.7625" width="1.016" layer="16"/>
+<wire x1="96.52" y1="1.27" x2="96.52" y2="1.905" width="1.016" layer="16"/>
+<wire x1="96.52" y1="1.905" x2="96.52" y2="2.54" width="1.016" layer="16"/>
 <wire x1="94.615" y1="4.7625" x2="85.725" y2="4.7625" width="1.016" layer="16"/>
-<wire x1="85.725" y1="4.7625" x2="79.375" y2="10.795" width="1.016" layer="16"/>
-<wire x1="79.375" y1="10.795" x2="76.2" y2="10.795" width="1.016" layer="16"/>
 <wire x1="76.2" y1="10.795" x2="75.565" y2="11.43" width="1.016" layer="16"/>
 <wire x1="75.565" y1="11.43" x2="69.215" y2="11.43" width="1.016" layer="16"/>
+<wire x1="76.2" y1="10.795" x2="79.6925" y2="10.795" width="1.016" layer="16"/>
+<wire x1="79.6925" y1="10.795" x2="85.725" y2="4.7625" width="1.016" layer="16"/>
+<wire x1="94.615" y1="4.7625" x2="96.52" y2="2.8575" width="1.016" layer="16"/>
+<wire x1="96.52" y1="2.8575" x2="96.52" y2="2.54" width="1.016" layer="16"/>
 </signal>
 <signal name="N$40">
@@
 <contactref element="R28" pad="2"/>
 <contactref element="R32" pad="1"/>
-<wire x1="58.42" y1="22.86" x2="58.42" y2="26.035" width="1.016" layer="16"/>
-<wire x1="58.42" y1="26.035" x2="62.23" y2="30.48" width="1.016" layer="16"/>
-<wire x1="62.23" y1="30.48" x2="62.23" y2="36.83" width="1.016" layer="16"/>
+<wire x1="62.23" y1="29.845" x2="62.23" y2="36.83" width="1.016" layer="16"/>
+<wire x1="62.23" y1="29.845" x2="58.42" y2="26.035" width="1.016" layer="16"/>
+<wire x1="58.42" y1="26.035" x2="58.42" y2="22.86" width="1.016" layer="16"/>
 </signal>
 <signal name="N$23">
@@
 <wire x1="52.07" y1="34.29" x2="52.07" y2="41.91" width="1.016" layer="16"/>
 <wire x1="41.91" y1="34.29" x2="44.45" y2="34.29" width="1.016" layer="16"/>
-<wire x1="49.53" y1="35.56" x2="49.53" y2="34.29" width="1.016" layer="16"/>
 <wire x1="49.53" y1="34.29" x2="52.07" y2="34.29" width="1.016" layer="16"/>
 <wire x1="50.8" y1="25.4" x2="50.8" y2="24.13" width="1.016" layer="16"/>
@@
 <wire x1="44.45" y1="34.29" x2="44.45" y2="36.83" width="1.016" layer="16"/>
 <wire x1="44.45" y1="36.83" x2="45.72" y2="38.1" width="1.016" layer="16"/>
-<wire x1="45.72" y1="38.1" x2="47.625" y2="38.1" width="1.016" layer="16"/>
-<wire x1="47.625" y1="38.1" x2="49.53" y2="35.56" width="1.016" layer="16"/>
+<wire x1="49.53" y1="34.29" x2="49.53" y2="36.83" width="1.016" layer="16"/>
+<wire x1="49.53" y1="36.83" x2="48.26" y2="38.1" width="1.016" layer="16"/>
+<wire x1="48.26" y1="38.1" x2="45.72" y2="38.1" width="1.016" layer="16"/>
 </signal>
 <signal name="N$45">
@@
 <wire x1="81.28" y1="49.53" x2="80.645" y2="48.895" width="1.016" layer="16"/>
 <wire x1="80.645" y1="48.895" x2="59.69" y2="48.895" width="1.016" layer="16"/>
-<wire x1="59.69" y1="48.895" x2="55.88" y2="45.72" width="1.016" layer="16"/>
-<wire x1="55.88" y1="45.72" x2="54.61" y2="44.45" width="1.016" layer="16"/>
-<wire x1="54.61" y1="44.45" x2="54.61" y2="41.91" width="1.016" layer="16"/>
+<wire x1="54.61" y1="41.91" x2="54.61" y2="43.815" width="1.016" layer="16"/>
+<wire x1="54.61" y1="43.815" x2="59.69" y2="48.895" width="1.016" layer="16"/>
 </signal>
 <signal name="MUX1*A">
