File: minipro4/Teilentwurf.sch (EAGLE design)
At the start: 89 parts, among them IC1 MEGA8-P, IC2 FT232RL_ADAPTER, IC3 78L08Z, IC4 4051N, IC5 TL082P, IC6 4051N, IC7 TL082P, J1 HOHLSTECKER, Q2 BS170, Q3 BS170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

Commit message: eagle iteration
Connections:
- net GND: now also C20.2, C21.1, C22.2, C23.1, C24.2, C25.1, IC4P.GND, IC6P.GND
- net V+: now also C20.1, C22.1, C24.1, IC4P.V+, IC6P.V+, IC7P.V+
- net V-: now also C21.2, C23.2, C25.2, IC4P.V-, IC6P.V-, IC7P.V-
Other:
- moved on the sheet: C18, C19, C20, C21, C24, C25
Changed lines of the file:
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@@
 <part name="P+5" library="03_device-library" deviceset="V+" device=""/>
 <part name="P-3" library="03_device-library" deviceset="V-" device=""/>
+<part name="P+8" library="03_device-library" deviceset="V+" device=""/>
+<part name="P+9" library="03_device-library" deviceset="V+" device=""/>
+<part name="P+12" library="03_device-library" deviceset="V+" device=""/>
+<part name="P-4" library="03_device-library" deviceset="V-" device=""/>
+<part name="P-5" library="03_device-library" deviceset="V-" device=""/>
+<part name="P-6" library="03_device-library" deviceset="V-" device=""/>
+<part name="GND19" library="03_device-library" deviceset="GND" device=""/>
+<part name="GND20" library="03_device-library" deviceset="GND" device=""/>
+<part name="GND21" library="03_device-library" deviceset="GND" device=""/>
 </parts>
 <sheets>
@@
 <instance part="C17" gate="G$1" x="355.6" y="-35.56"/>
 <instance part="GND17" gate="1" x="355.6" y="-48.26"/>
-<instance part="C18" gate="G$1" x="304.8" y="73.66"/>
-<instance part="C19" gate="G$1" x="304.8" y="58.42"/>
-<instance part="C20" gate="G$1" x="330.2" y="76.2"/>
-<instance part="C21" gate="G$1" x="332.74" y="60.96"/>
+<instance part="C18" gate="G$1" x="287.02" y="73.66"/>
+<instance part="C19" gate="G$1" x="287.02" y="58.42"/>
+<instance part="C20" gate="G$1" x="327.66" y="71.12"/>
+<instance part="C21" gate="G$1" x="327.66" y="60.96"/>
 <instance part="C22" gate="G$1" x="358.14" y="73.66"/>
 <instance part="C23" gate="G$1" x="355.6" y="60.96"/>
-<instance part="C24" gate="G$1" x="378.46" y="73.66"/>
-<instance part="C25" gate="G$1" x="373.38" y="58.42"/>
-<instance part="IC5" gate="P" x="294.64" y="63.5"/>
-<instance part="IC7" gate="P" x="322.58" y="66.04"/>
+<instance part="C24" gate="G$1" x="396.24" y="73.66"/>
+<instance part="C25" gate="G$1" x="396.24" y="55.88"/>
+<instance part="IC5" gate="P" x="276.86" y="63.5"/>
+<instance part="IC7" gate="P" x="317.5" y="66.04"/>
 <instance part="IC6" gate="P" x="347.98" y="66.04"/>
 <instance part="IC4" gate="P" x="388.62" y="66.04"/>
-<instance part="GND18" gate="1" x="309.88" y="60.96"/>
-<instance part="P+5" gate="1" x="304.8" y="83.82"/>
-<instance part="P-3" gate="1" x="304.8" y="43.18"/>
+<instance part="GND18" gate="1" x="292.1" y="60.96"/>
+<instance part="P+5" gate="1" x="287.02" y="83.82"/>
+<instance part="P-3" gate="1" x="287.02" y="43.18"/>
+<instance part="P+8" gate="1" x="317.5" y="83.82"/>
+<instance part="P+9" gate="1" x="347.98" y="86.36"/>
+<instance part="P+12" gate="1" x="393.7" y="86.36"/>
+<instance part="P-4" gate="1" x="327.66" y="45.72"/>
+<instance part="P-5" gate="1" x="355.6" y="45.72"/>
+<instance part="P-6" gate="1" x="391.16" y="45.72"/>
+<instance part="GND19" gate="1" x="335.28" y="60.96"/>
+<instance part="GND20" gate="1" x="365.76" y="60.96"/>
+<instance part="GND21" gate="1" x="403.86" y="58.42"/>
 </instances>
 <busses>
@@
 <pinref part="C18" gate="G$1" pin="2"/>
 <pinref part="C19" gate="G$1" pin="1"/>
-<wire x1="304.8" y1="68.58" x2="304.8" y2="66.04" width="0.1524" layer="91"/>
-<wire x1="304.8" y1="66.04" x2="304.8" y2="60.96" width="0.1524" layer="91"/>
-<wire x1="304.8" y1="66.04" x2="309.88" y2="66.04" width="0.1524" layer="91"/>
-<wire x1="309.88" y1="66.04" x2="309.88" y2="63.5" width="0.1524" layer="91"/>
-<junction x="304.8" y="66.04"/>
+<wire x1="287.02" y1="68.58" x2="287.02" y2="66.04" width="0.1524" layer="91"/>
+<wire x1="287.02" y1="66.04" x2="287.02" y2="60.96" width="0.1524" layer="91"/>
+<wire x1="287.02" y1="66.04" x2="292.1" y2="66.04" width="0.1524" layer="91"/>
+<wire x1="292.1" y1="66.04" x2="292.1" y2="63.5" width="0.1524" layer="91"/>
+<junction x="287.02" y="66.04"/>
 <pinref part="GND18" gate="1" pin="GND"/>
+</segment>
+<segment>
+<pinref part="C20" gate="G$1" pin="2"/>
+<pinref part="C21" gate="G$1" pin="1"/>
+<wire x1="327.66" y1="66.04" x2="327.66" y2="63.5" width="0.1524" layer="91"/>
+<pinref part="GND19" gate="1" pin="GND"/>
+<wire x1="335.28" y1="63.5" x2="327.66" y2="63.5" width="0.1524" layer="91"/>
+<junction x="327.66" y="63.5"/>
+</segment>
+<segment>
+<pinref part="IC6" gate="P" pin="GND"/>
+<wire x1="347.98" y1="58.42" x2="350.52" y2="58.42" width="0.1524" layer="91"/>
+<wire x1="350.52" y1="58.42" x2="350.52" y2="63.5" width="0.1524" layer="91"/>
+<pinref part="C23" gate="G$1" pin="1"/>
+<wire x1="350.52" y1="63.5" x2="355.6" y2="63.5" width="0.1524" layer="91"/>
+<pinref part="C22" gate="G$1" pin="2"/>
+<wire x1="358.14" y1="68.58" x2="355.6" y2="68.58" width="0.1524" layer="91"/>
+<wire x1="355.6" y1="68.58" x2="355.6" y2="63.5" width="0.1524" layer="91"/>
+<junction x="355.6" y="63.5"/>
+<pinref part="GND20" gate="1" pin="GND"/>
+<wire x1="365.76" y1="63.5" x2="355.6" y2="63.5" width="0.1524" layer="91"/>
+</segment>
+<segment>
+<pinref part="C25" gate="G$1" pin="1"/>
+<pinref part="C24" gate="G$1" pin="2"/>
+<wire x1="396.24" y1="58.42" x2="396.24" y2="60.96" width="0.1524" layer="91"/>
+<pinref part="IC4" gate="P" pin="GND"/>
+<wire x1="396.24" y1="60.96" x2="396.24" y2="68.58" width="0.1524" layer="91"/>
+<wire x1="388.62" y1="58.42" x2="396.24" y2="58.42" width="0.1524" layer="91"/>
+<junction x="396.24" y="58.42"/>
+<pinref part="GND21" gate="1" pin="GND"/>
+<wire x1="403.86" y1="60.96" x2="396.24" y2="60.96" width="0.1524" layer="91"/>
+<junction x="396.24" y="60.96"/>
 </segment>
 </net>
@@
 <segment>
 <pinref part="C18" gate="G$1" pin="1"/>
-<wire x1="304.8" y1="76.2" x2="304.8" y2="78.74" width="0.1524" layer="91"/>
+<wire x1="287.02" y1="76.2" x2="287.02" y2="78.74" width="0.1524" layer="91"/>
 <pinref part="IC5" gate="P" pin="V+"/>
-<wire x1="304.8" y1="78.74" x2="294.64" y2="78.74" width="0.1524" layer="91"/>
-<wire x1="294.64" y1="78.74" x2="294.64" y2="71.12" width="0.1524" layer="91"/>
-<wire x1="304.8" y1="78.74" x2="304.8" y2="81.28" width="0.1524" layer="91"/>
-<junction x="304.8" y="78.74"/>
+<wire x1="287.02" y1="78.74" x2="276.86" y2="78.74" width="0.1524" layer="91"/>
+<wire x1="276.86" y1="78.74" x2="276.86" y2="71.12" width="0.1524" layer="91"/>
+<wire x1="287.02" y1="78.74" x2="287.02" y2="81.28" width="0.1524" layer="91"/>
+<junction x="287.02" y="78.74"/>
 <pinref part="P+5" gate="1" pin="V+"/>
+</segment>
+<segment>
+<pinref part="IC7" gate="P" pin="V+"/>
+<wire x1="317.5" y1="73.66" x2="317.5" y2="81.28" width="0.1524" layer="91"/>
+<wire x1="317.5" y1="81.28" x2="327.66" y2="81.28" width="0.1524" layer="91"/>
+<pinref part="C20" gate="G$1" pin="1"/>
+<wire x1="327.66" y1="81.28" x2="327.66" y2="73.66" width="0.1524" layer="91"/>
+<pinref part="P+8" gate="1" pin="V+"/>
+<junction x="317.5" y="81.28"/>
+</segment>
+<segment>
+<pinref part="C22" gate="G$1" pin="1"/>
+<wire x1="358.14" y1="76.2" x2="358.14" y2="83.82" width="0.1524" layer="91"/>
+<pinref part="IC6" gate="P" pin="V+"/>
+<wire x1="358.14" y1="83.82" x2="347.98" y2="83.82" width="0.1524" layer="91"/>
+<wire x1="347.98" y1="83.82" x2="347.98" y2="73.66" width="0.1524" layer="91"/>
+<pinref part="P+9" gate="1" pin="V+"/>
+<junction x="347.98" y="83.82"/>
+</segment>
+<segment>
+<pinref part="C24" gate="G$1" pin="1"/>
+<wire x1="396.24" y1="76.2" x2="396.24" y2="83.82" width="0.1524" layer="91"/>
+<pinref part="IC4" gate="P" pin="V+"/>
+<wire x1="396.24" y1="83.82" x2="393.7" y2="83.82" width="0.1524" layer="91"/>
+<wire x1="393.7" y1="83.82" x2="388.62" y2="83.82" width="0.1524" layer="91"/>
+<wire x1="388.62" y1="83.82" x2="388.62" y2="73.66" width="0.1524" layer="91"/>
+<pinref part="P+12" gate="1" pin="V+"/>
+<junction x="393.7" y="83.82"/>
 </segment>
 </net>
@@
 <segment>
 <pinref part="IC5" gate="P" pin="V-"/>
-<wire x1="294.64" y1="55.88" x2="294.64" y2="48.26" width="0.1524" layer="91"/>
+<wire x1="276.86" y1="55.88" x2="276.86" y2="48.26" width="0.1524" layer="91"/>
 <pinref part="C19" gate="G$1" pin="2"/>
-<wire x1="294.64" y1="48.26" x2="304.8" y2="48.26" width="0.1524" layer="91"/>
-<wire x1="304.8" y1="48.26" x2="304.8" y2="53.34" width="0.1524" layer="91"/>
-<wire x1="304.8" y1="48.26" x2="304.8" y2="45.72" width="0.1524" layer="91"/>
-<junction x="304.8" y="48.26"/>
+<wire x1="276.86" y1="48.26" x2="287.02" y2="48.26" width="0.1524" layer="91"/>
+<wire x1="287.02" y1="48.26" x2="287.02" y2="53.34" width="0.1524" layer="91"/>
+<wire x1="287.02" y1="48.26" x2="287.02" y2="45.72" width="0.1524" layer="91"/>
+<junction x="287.02" y="48.26"/>
 <pinref part="P-3" gate="1" pin="V-"/>
 </segment>
+<segment>
+<pinref part="C21" gate="G$1" pin="2"/>
+<wire x1="327.66" y1="55.88" x2="327.66" y2="48.26" width="0.1524" layer="91"/>
+<pinref part="IC7" gate="P" pin="V-"/>
+<wire x1="327.66" y1="48.26" x2="317.5" y2="48.26" width="0.1524" layer="91"/>
+<wire x1="317.5" y1="48.26" x2="317.5" y2="58.42" width="0.1524" layer="91"/>
+<pinref part="P-4" gate="1" pin="V-"/>
+<junction x="327.66" y="48.26"/>
+</segment>
+<segment>
+<pinref part="IC6" gate="P" pin="V-"/>
+<wire x1="342.9" y1="58.42" x2="342.9" y2="48.26" width="0.1524" layer="91"/>
+<pinref part="C23" gate="G$1" pin="2"/>
+<wire x1="342.9" y1="48.26" x2="355.6" y2="48.26" width="0.1524" layer="91"/>
+<wire x1="355.6" y1="48.26" x2="355.6" y2="55.88" width="0.1524" layer="91"/>
+<pinref part="P-5" gate="1" pin="V-"/>
+<junction x="355.6" y="48.26"/>
+</segment>
+<segment>
+<pinref part="IC4" gate="P" pin="V-"/>
+<wire x1="383.54" y1="58.42" x2="383.54" y2="48.26" width="0.1524" layer="91"/>
+<pinref part="C25" gate="G$1" pin="2"/>
+<wire x1="383.54" y1="48.26" x2="391.16" y2="48.26" width="0.1524" layer="91"/>
+<wire x1="391.16" y1="48.26" x2="396.24" y2="48.26" width="0.1524" layer="91"/>
+<wire x1="396.24" y1="48.26" x2="396.24" y2="50.8" width="0.1524" layer="91"/>
+<pinref part="P-6" gate="1" pin="V-"/>
+<junction x="391.16" y="48.26"/>
+</segment>
 </net>

Commit message: Layout
Parts:
- added R33: 0, 03_device-library:R-EU_0207/10
- R28, R32: device 03_device-library:R-EU_0207/10 -> 03_device-library:R-EU_0207/15
Connections:
- new net N$42: IC6A.C, R33.2
- net MUX2*: now also R33.1; no longer IC6A.C
- net N$25: now also IC5B.+IN; no longer IC5A.+IN
- net N$26: now also IC5B.-IN; no longer IC5A.-IN
- net N$27: now also IC5A.+IN; no longer IC5B.+IN
- net N$34: now also IC5B.OUT; no longer IC5A.OUT
- net N$35: now also IC5A.OUT; no longer IC5B.OUT
- net N$36: now also IC5A.-IN; no longer IC5B.-IN
Other:
- moved on the sheet: IC5A, IC5B
Changed lines of the file:
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@@
 <part name="R26" library="03_device-library" deviceset="POT" device="" value="100k"/>
 <part name="R27" library="03_device-library" deviceset="R-EU_" device="0207/10" value="22k"/>
-<part name="R28" library="03_device-library" deviceset="R-EU_" device="0207/10" value="8k2"/>
-<part name="R32" library="03_device-library" deviceset="R-EU_" device="0207/10" value="220"/>
+<part name="R28" library="03_device-library" deviceset="R-EU_" device="0207/15" value="8k2"/>
+<part name="R32" library="03_device-library" deviceset="R-EU_" device="0207/15" value="220"/>
 <part name="C17" library="03_device-library" deviceset="C-EU" device="025-030X050" value="1nF"/>
 <part name="GND17" library="03_device-library" deviceset="GND" device=""/>
@@
 <part name="GND20" library="03_device-library" deviceset="GND" device=""/>
 <part name="GND21" library="03_device-library" deviceset="GND" device=""/>
+<part name="R33" library="03_device-library" deviceset="R-EU_" device="0207/10" value="0"/>
 </parts>
 <sheets>
@@
 <instance part="GND12" gate="1" x="-2.54" y="-20.32"/>
 <instance part="GND13" gate="1" x="78.74" y="-60.96"/>
-<instance part="IC5" gate="A" x="162.56" y="-30.48"/>
-<instance part="IC5" gate="B" x="256.54" y="-27.94"/>
+<instance part="IC5" gate="B" x="162.56" y="-30.48"/>
+<instance part="IC5" gate="A" x="256.54" y="-27.94"/>
 <instance part="IC6" gate="A" x="144.78" y="-63.5" rot="MR0"/>
 <instance part="R15" gate="G$1" x="198.12" y="-88.9" rot="R90"/>
@@
 <instance part="GND20" gate="1" x="365.76" y="60.96"/>
 <instance part="GND21" gate="1" x="403.86" y="58.42"/>
+<instance part="R33" gate="G$1" x="160.02" y="-86.36" rot="R90"/>
 </instances>
 <busses>
@@
 </segment>
 <segment>
-<pinref part="IC6" gate="A" pin="C"/>
-<wire x1="157.48" y1="-78.74" x2="160.02" y2="-78.74" width="0.1524" layer="91"/>
-<wire x1="160.02" y1="-78.74" x2="160.02" y2="-93.98" width="0.1524" layer="91"/>
-<label x="160.02" y="-78.74" size="1.778" layer="95"/>
+<pinref part="R33" gate="G$1" pin="1"/>
+<wire x1="160.02" y1="-91.44" x2="160.02" y2="-93.98" width="0.1524" layer="91"/>
+<label x="160.02" y="-101.6" size="1.778" layer="95"/>
 </segment>
 </net>
@@
 <segment>
 <pinref part="IC4" gate="A" pin="X"/>
-<pinref part="IC5" gate="A" pin="+IN"/>
+<pinref part="IC5" gate="B" pin="+IN"/>
 <wire x1="119.38" y1="-15.24" x2="154.94" y2="-15.24" width="0.1524" layer="91"/>
 <wire x1="154.94" y1="-15.24" x2="154.94" y2="-27.94" width="0.1524" layer="91"/>
@@
 <pinref part="IC6" gate="A" pin="X"/>
 <wire x1="132.08" y1="-48.26" x2="132.08" y2="-35.56" width="0.1524" layer="91"/>
-<pinref part="IC5" gate="A" pin="-IN"/>
+<pinref part="IC5" gate="B" pin="-IN"/>
 <wire x1="132.08" y1="-35.56" x2="154.94" y2="-35.56" width="0.1524" layer="91"/>
 <wire x1="154.94" y1="-35.56" x2="154.94" y2="-33.02" width="0.1524" layer="91"/>
@@
 <net name="N$34" class="0">
 <segment>
-<pinref part="IC5" gate="A" pin="OUT"/>
+<pinref part="IC5" gate="B" pin="OUT"/>
 <pinref part="R16" gate="G$1" pin="2"/>
 <wire x1="170.18" y1="-30.48" x2="198.12" y2="-30.48" width="0.1524" layer="91"/>
@@
 <wire x1="236.22" y1="-25.4" x2="248.92" y2="-25.4" width="0.1524" layer="91"/>
 <junction x="236.22" y="-25.4"/>
-<pinref part="IC5" gate="B" pin="+IN"/>
+<pinref part="IC5" gate="A" pin="+IN"/>
 </segment>
 </net>
 <net name="N$35" class="0">
 <segment>
-<pinref part="IC5" gate="B" pin="OUT"/>
+<pinref part="IC5" gate="A" pin="OUT"/>
 <wire x1="264.16" y1="-27.94" x2="276.86" y2="-27.94" width="0.1524" layer="91"/>
 <pinref part="R24" gate="G$1" pin="1"/>
@@
 <net name="N$36" class="0">
 <segment>
-<pinref part="IC5" gate="B" pin="-IN"/>
+<pinref part="IC5" gate="A" pin="-IN"/>
 <wire x1="248.92" y1="-30.48" x2="248.92" y2="-40.64" width="0.1524" layer="91"/>
 <wire x1="248.92" y1="-40.64" x2="266.7" y2="-40.64" width="0.1524" layer="91"/>
@@
 </segment>
 </net>
+<net name="N$42" class="0">
+<segment>
+<pinref part="IC6" gate="A" pin="C"/>
+<wire x1="157.48" y1="-78.74" x2="160.02" y2="-78.74" width="0.1524" layer="91"/>
+<pinref part="R33" gate="G$1" pin="2"/>
+<wire x1="160.02" y1="-78.74" x2="160.02" y2="-81.28" width="0.1524" layer="91"/>
+</segment>
+</net>

Commit message: Layout Iteration
Parts:
- added R34: 0, 03_device-library:R-EU_0207/10
- R25: device 03_device-library:R-EU_0207/10 -> resistor:R-EU_0207/7
- R28: device 03_device-library:R-EU_0207/15 -> 03_device-library:R-EU_0207/10
Connections:
- removed net N$42: IC6A.C, R33.2
- new net MUX1*A: IC4A.B, R33.1
- new net N$45: IC6A.A, R34.2
- net MUX0*: now also R34.1; no longer IC6A.A
- net MUX1*: now also R33.2; no longer IC4A.B
- net MUX2*: now also IC6A.C; no longer R33.1
Other:
- moved on the sheet: R33
Changed lines of the file:
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@@
 <part name="GND16" library="03_device-library" deviceset="GND" device=""/>
 <part name="IC7" library="03_device-library" deviceset="TL082" device="P"/>
-<part name="R25" library="03_device-library" deviceset="R-EU_" device="0207/10" value="100k"/>
+<part name="R25" library="resistor" deviceset="R-EU_" device="0207/7" value="100k"/>
 <part name="P+4" library="03_device-library" deviceset="V+" device=""/>
 <part name="P-2" library="03_device-library" deviceset="V-" device=""/>
 <part name="R26" library="03_device-library" deviceset="POT" device="" value="100k"/>
 <part name="R27" library="03_device-library" deviceset="R-EU_" device="0207/10" value="22k"/>
-<part name="R28" library="03_device-library" deviceset="R-EU_" device="0207/15" value="8k2"/>
+<part name="R28" library="03_device-library" deviceset="R-EU_" device="0207/10" value="8k2"/>
 <part name="R32" library="03_device-library" deviceset="R-EU_" device="0207/15" value="220"/>
 <part name="C17" library="03_device-library" deviceset="C-EU" device="025-030X050" value="1nF"/>
@@
 <part name="GND21" library="03_device-library" deviceset="GND" device=""/>
 <part name="R33" library="03_device-library" deviceset="R-EU_" device="0207/10" value="0"/>
+<part name="R34" library="03_device-library" deviceset="R-EU_" device="0207/10" value="0"/>
 </parts>
 <sheets>
@@
 <instance part="GND20" gate="1" x="365.76" y="60.96"/>
 <instance part="GND21" gate="1" x="403.86" y="58.42"/>
-<instance part="R33" gate="G$1" x="160.02" y="-86.36" rot="R90"/>
+<instance part="R33" gate="G$1" x="165.1" y="-83.82" rot="R90"/>
+<instance part="R34" gate="G$1" x="167.64" y="-88.9" rot="R90"/>
 </instances>
 <busses>
@@
 </segment>
 <segment>
-<pinref part="IC6" gate="A" pin="A"/>
-<wire x1="157.48" y1="-73.66" x2="170.18" y2="-73.66" width="0.1524" layer="91"/>
-<wire x1="170.18" y1="-73.66" x2="170.18" y2="-93.98" width="0.1524" layer="91"/>
-<label x="160.02" y="-73.66" size="1.778" layer="95"/>
+<pinref part="R34" gate="G$1" pin="1"/>
+<wire x1="167.64" y1="-93.98" x2="167.64" y2="-106.68" width="0.1524" layer="91"/>
+<label x="162.56" y="-109.22" size="1.778" layer="95"/>
 </segment>
 </net>
@@
 </segment>
 <segment>
-<pinref part="R33" gate="G$1" pin="1"/>
-<wire x1="160.02" y1="-91.44" x2="160.02" y2="-93.98" width="0.1524" layer="91"/>
-<label x="160.02" y="-101.6" size="1.778" layer="95"/>
+<pinref part="IC6" gate="A" pin="C"/>
+<wire x1="157.48" y1="-78.74" x2="157.48" y2="-99.06" width="0.1524" layer="91"/>
+<label x="157.48" y="-99.06" size="1.778" layer="95"/>
 </segment>
 </net>
@@
 </segment>
 <segment>
-<pinref part="IC4" gate="A" pin="B"/>
-<wire x1="93.98" y1="-43.18" x2="88.9" y2="-43.18" width="0.1524" layer="91"/>
-<label x="91.44" y="-43.18" size="1.778" layer="95"/>
-</segment>
-<segment>
 <pinref part="IC6" gate="A" pin="B"/>
+<pinref part="R33" gate="G$1" pin="2"/>
 <wire x1="157.48" y1="-76.2" x2="165.1" y2="-76.2" width="0.1524" layer="91"/>
-<wire x1="165.1" y1="-76.2" x2="165.1" y2="-93.98" width="0.1524" layer="91"/>
-<label x="160.02" y="-76.2" size="1.778" layer="95"/>
+<wire x1="165.1" y1="-76.2" x2="165.1" y2="-78.74" width="0.1524" layer="91"/>
 </segment>
 </net>
@@
 </segment>
 </net>
-<net name="N$42" class="0">
-<segment>
-<pinref part="IC6" gate="A" pin="C"/>
-<wire x1="157.48" y1="-78.74" x2="160.02" y2="-78.74" width="0.1524" layer="91"/>
-<pinref part="R33" gate="G$1" pin="2"/>
-<wire x1="160.02" y1="-78.74" x2="160.02" y2="-81.28" width="0.1524" layer="91"/>
-</segment>
-</net>
+<net name="N$45" class="0">
+<segment>
+<pinref part="IC6" gate="A" pin="A"/>
+<pinref part="R34" gate="G$1" pin="2"/>
+<wire x1="157.48" y1="-73.66" x2="167.64" y2="-73.66" width="0.1524" layer="91"/>
+<wire x1="167.64" y1="-73.66" x2="167.64" y2="-83.82" width="0.1524" layer="91"/>
+</segment>
+</net>
+<net name="MUX1*A" class="0">
+<segment>
+<pinref part="R33" gate="G$1" pin="1"/>
+<wire x1="165.1" y1="-88.9" x2="165.1" y2="-99.06" width="0.1524" layer="91"/>
+<label x="165.1" y="-96.52" size="1.778" layer="95"/>
+</segment>
+<segment>
+<pinref part="IC4" gate="A" pin="B"/>
+<wire x1="93.98" y1="-43.18" x2="88.9" y2="-43.18" width="0.1524" layer="91"/>
+<label x="91.44" y="-43.18" size="1.778" layer="95"/>
+</segment>
+</net>
